Commit message: robot goes down to grip, added force sensor but force equal to zero all the time

File: panda_arm.urdf (robot description, URDF)
Before this commit: robot panda_arm, 8 links, 7 joints
Links:
- link link7: geometry collision mesh filename=../../../model/panda/meshes/collision/hand.obj; collision mesh filename=../../../model/panda/meshes/collision/link7.obj

File: panda_arm_hand.urdf (robot description, URDF)
Before this commit: robot panda_arm_hand, 10 links, 9 joints
Links:
- link link7: geometry collision mesh filename=../../../model/panda/meshes/collision/hand.obj; collision mesh filename=../../../model/panda/meshes/collision/link7.obj
