Commit message: Made a separate urdf for the visualization that has a hand. Controller does not use the hand urdf. Currently errors due to OTG goalPositionAndVelocity

File: panda_arm_hand.urdf (robot description, URDF)
Before this commit: robot panda_arm, 8 links, 7 joints
Links:
- added link leftfinger, mass 0.1; visual mesh filename=../../../model/panda/meshes/visual/finger.obj
- added link rightfinger, mass 0.1; visual mesh filename=../../../model/panda/meshes/visual/finger.obj
Joints:
- added joint finger_joint1: type prismatic, parent link7, child leftfinger, origin xyz=0 0 0.1654 rpy=0 0 -0.78539816339, axis 0 1 0, limit lower=0.0 upper=0.04 effort=20 velocity=0.2
- added joint finger_joint2: type prismatic, parent link7, child rightfinger, origin xyz=0 0 0.1654 rpy=0 0 -0.78539816339, axis 0 1 0, limit lower=0.0 upper=0.04 effort=20 velocity=0.2

Commit message: Added new fingers to the gripper

File: panda_arm_hand.urdf (robot description, URDF)
Before this commit: robot panda_arm_hand, 10 links, 9 joints
Links:
- link leftfinger: geometry collision mesh filename=../../../model/final_project/meshes/collision/gripper.obj; visual mesh filename=../../../model/final_project/meshes/collision/gripper.obj
- link rightfinger: geometry collision mesh filename=../../../model/final_project/meshes/collision/gripper.obj; visual mesh filename=../../../model/final_project/meshes/collision/gripper.obj

Commit message: Fixed the 35/45 degree offset problem

File: panda_arm_hand.urdf (robot description, URDF)
Before this commit: robot panda_arm_hand, 10 links, 9 joints
Joints:
- joint finger_joint1: origin xyz=0 0 0.1654 rpy=0 0 -0.78539816339 -> xyz=0 0 0.1654 rpy=0 0 0
- joint finger_joint2: origin xyz=0 0 0.1654 rpy=0 0 -0.78539816339 -> xyz=0 0 0.1654 rpy=0 0 0

Commit message: Updated visuals to add walls, soft gripper, thigh and longer footlink, colored table, etc

File: panda_arm_hand.urdf (robot description, URDF)
Before this commit: robot panda_arm_hand, 10 links, 9 joints
Links:
- link leftfinger: geometry collision mesh filename=../../../model/final_project/meshes/collision/gripper.obj; visual mesh filename=../../../model/final_project/meshes/visual/gripper_soft.obj
- link rightfinger: geometry collision mesh filename=../../../model/final_project/meshes/collision/gripper.obj; visual mesh filename=../../../model/final_project/meshes/visual/gripper_soft.obj

Commit message: Added the chunky gripper, made it pinkish, tried to keep the robot from dropping the leg too far from the ground at the end

File: panda_arm_hand.urdf (robot description, URDF)
Before this commit: robot panda_arm_hand, 10 links, 9 joints
Links:
- link leftfinger: geometry collision mesh filename=../../../model/final_project/meshes/collision/gripper.obj; visual mesh filename=../../../model/final_project/meshes/visual/chunky_gripper.o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
- link rightfinger: geometry collision mesh filename=../../../model/final_project/meshes/collision/gripper.obj; visual mesh filename=../../../model/final_project/meshes/visual/chunky_gripper.o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
