Commit message: leg working after William and Adrian OH

File: human_leg.urdf (robot description, URDF)
Before this commit: robot leg, 3 links, 2 joints
Links:
- link link0: geometry visual mesh filename=../../../model/panda/meshes/visual/link0.obj
- link link2: geometry collision cylinder length=0.5 radius=0.05; visual cylinder length=0.5 radius=0.05
Joints:
- joint joint1: origin xyz=0 0 0 rpy=0 -1.57079632679 0 -> xyz=0 0 0 rpy=0 0 0
- joint joint2: origin xyz=0 0 0 rpy=0 0 0 -> xyz=0 0 0.5 rpy=0 0 0

Commit message: workiiing

File: human_leg.urdf (robot description, URDF)
Before this commit: robot leg, 3 links, 2 joints
Links:
- link link1: mass 4 -> 1
- link link2: mass 3 -> 1
Joints:
- joint joint2: limit lower=-1.7628 upper=1.7628 effort=87 velocity=2.1750 -> lower=-1.7628 upper=-0.61 effort=87 velocity=2.1750

File: panda_arm_hand.urdf (robot description, URDF)
Before this commit: robot panda_arm_hand, 10 links, 9 joints
Joints:
- joint finger_joint1: limit lower=0.0 upper=0.04 effort=20 velocity=0.2 -> lower=0.0 upper=0.15 effort=500 velocity=0.2
- joint finger_joint2: limit lower=0.0 upper=0.04 effort=20 velocity=0.2 -> lower=0.0 upper=0.15 effort=500 velocity=0.2

Commit message: not slipping

File: human_leg.urdf (robot description, URDF)
Before this commit: robot leg, 3 links, 2 joints
Links:
- link link2: geometry collision cylinder length=0.5 radius=0.05; visual mesh filename=../../../model/final_project/meshes/visual/footlink.obj

Commit message: remove the visual spheres and forces

File: human_leg.urdf (robot description, URDF)
Before this commit: robot leg, 3 links, 2 joints
Links:
- link link1: geometry collision cylinder length=0.5 radius=0.05; visual cylinder length=0.5 radius=0.05
- link link2: geometry collision cylinder length=0.5 radius=0.05; visual mesh filename=../../../model/final_project/meshes/visual/footlink.obj

Commit message: Lots of cad and mtl files. Also made the sim a bit faster - changes 6/100 to 6/50

File: human_leg.urdf (robot description, URDF)
Before this commit: robot leg, 3 links, 2 joints
Links:
- link link1: geometry collision cylinder length=0.5 radius=0.05; visual mesh filename=../../../model/final_project/meshes/visual/long_thigh.obj
- link link2: geometry collision cylinder length=0.5 radius=0.05; visual mesh filename=../../../model/final_project/meshes/visual/long_footlink.obj

Commit message: change colors and link0

File: human_leg.urdf (robot description, URDF)
Before this commit: robot leg, 3 links, 2 joints
Links:
- link link0: geometry 

File: human_leg_right.urdf (robot description, URDF)
Before this commit: robot right_leg, 3 links, 2 joints
Links:
- link link0: geometry 

Commit message: Rotated table, moved Robert a bit, made his knees colored the same as the rest of his body

File: human_leg.urdf (robot description, URDF)
Before this commit: robot leg, 3 links, 2 joints
Links:
- link link1: geometry collision cylinder length=0.5 radius=0.05; visual mesh filename=../../../model/final_project/meshes/visual/long_thigh.obj
- link link2: geometry collision cylinder length=0.5 radius=0.05; visual mesh filename=../../../model/final_project/meshes/visual/long_footlink.obj

File: human_leg_right.urdf (robot description, URDF)
Before this commit: robot right_leg, 3 links, 2 joints
Links:
- link link1: geometry collision cylinder length=0.5 radius=0.05; visual mesh filename=../../../model/final_project/meshes/visual/long_thigh.obj
- link link2: geometry collision cylinder length=0.5 radius=0.05; visual mesh filename=../../../model/final_project/meshes/visual/right_footlink.o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
